File: fuzz.brd (EAGLE design)
At the start: 100 x 70 mm, 19 parts, among them T1 2N3904, T2 2N3904

Commit message: 1.1
Parts:
- removed C1: 22uF, resistor:C025-024X044
- removed D1: 1N4004, diode:DO41-10
- removed GND, IN, IN2: (no value), pinhead:1X01
- removed JP3, JP5: (no value), pinhead:1X03
- added GROUND, INPUT1, INPUT2: (no value), wirepad:2,15/1,0
- added VOL1, VOL2: (no value), pinhead:1X03
- 9V: device pinhead:1X01 -> wirepad:2,15/1,0
- moved 9V 30.3 mm to (32.3, 17.9)
- moved T2 28.4 mm to (12.5, 15.8), turned to 270 degrees
- moved C5 24.6 mm to (24.8, 2.39), turned to 180 degrees
- moved D3 23.3 mm to (22.9, 10.5), turned to 180 degrees
- moved C3 22.1 mm to (26.4, 28.5), turned to 180 degrees
- moved C4 19.5 mm to (12.3, 9.42), turned to 270 degrees
- moved R3 14.3 mm to (2.26, 11.0)
- moved T1 14.0 mm to (15.3, 26.5), turned to 90 degrees
- moved D2 13.0 mm to (14.1, 21.5), turned to 0 degrees
- moved R2 10.7 mm to (24.2, 6.63), turned to 0 degrees
- moved R1 7.30 mm to (21.3, 23.4), turned to 270 degrees
- moved C2 6.09 mm to (9.09, 26.3)
Connections:
- removed net INPUT: C2.2, IN.1, R3.2
- removed net N$7: C5.1, IN2.1
- new net INPUT2: C5.2, INPUT2.1
- new net N$10: GROUND.1, R3.1, VOL2.3
- new net N$11: C2.1, D2.C
- net N$1: now also VOL1.1; no longer JP3.1
- net N$2: now also C2.2, INPUT1.1, R3.2; no longer C2.1, D2.C
- net N$4: now also C5.1, D3.C, T2.2; no longer 9V.1, C1.1, D1.C, R1.2, R2.2
- net N$6: now also 9V.1, R1.2, R2.2; no longer C5.2, D3.C, T2.2
- net N$8: now also VOL2.1; no longer JP5.1
- net N$9: now also VOL1.3; no longer C1.2, D1.A, GND.1, JP3.3, JP5.3, R3.1
Routing:
- net N$9: track 157.2 -> 31.6 mm
- net N$5: track 38.3 -> 14.9 mm
- net N$7: track 16.0 -> 0.00 mm
- net N$8: track 19.6 -> 5.43 mm
- net N$3: track 28.7 -> 17.6 mm
- net INPUT: track 10.4 -> 0.00 mm
- net N$6: track 17.4 -> 26.2 mm
- net N$10: track 0.00 -> 7.87 mm
- net N$4: track 33.5 -> 26.4 mm
- net INPUT2: track 0.00 -> 6.86 mm
- net N$11: track 0.00 -> 4.85 mm
- net N$1: track 1.06 -> 4.65 mm
